File: PCB/sensor-board-solar/sensor-board-solar.kicad_sch (KiCad schematic)
At the start: 7 parts, among them J1 Conn_01x02_Pin (Solar panel c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, U1 MAGNETIC POGO CONN., U2 MAGNETIC POGO CONN.

Commit message: Update PCB files (pressure + solar)#
Connections:
- net +3.3V: now also U1.1
- no-connect marks 1 -> 0
Changed lines of the file:
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@@
 		(color 0 0 0 0)
 	)
-	(no_connect
-		(at 149.86 68.58)
+	(junction
+		(at 173.99 64.77)
+		(diameter 0)
+		(color 0 0 0 0)
+	)
+	(junction
+		(at 154.94 68.58)
+		(diameter 0)
+		(color 0 0 0 0)
+	)
+	(wire
+		(pts
+			(xy 149.86 68.58) (xy 154.94 68.58)
+		)
+		(stroke
+			(width 0)
+			(type default)
+		)
 	)
 	(wire
@@
 	(wire
 		(pts
+			(xy 154.94 72.39) (xy 154.94 68.58)
+		)
+		(stroke
+			(width 0)
+			(type default)
+		)
+	)
+	(wire
+		(pts
 			(xy 85.09 82.55) (xy 85.09 83.82)
 		)
@@
 	(wire
 		(pts
+			(xy 173.99 64.77) (xy 173.99 72.39)
+		)
+		(stroke
+			(width 0)
+			(type default)
+		)
+	)
+	(wire
+		(pts
 			(xy 181.61 69.85) (xy 191.77 69.85)
 		)
@@
 	(wire
 		(pts
+			(xy 154.94 68.58) (xy 156.21 68.58)
+		)
+		(stroke
+			(width 0)
+			(type default)
+		)
+	)
+	(wire
+		(pts
 			(xy 85.09 69.85) (xy 85.09 73.66)
 		)
@@
 		(pts
 			(xy 87.63 95.25) (xy 87.63 92.71)
+		)
+		(stroke
+			(width 0)
+			(type default)
+		)
+	)
+	(wire
+		(pts
+			(xy 173.99 64.77) (xy 191.77 64.77)
+		)
+		(stroke
+			(width 0)
+			(type default)
+		)
+	)
+	(wire
+		(pts
+			(xy 173.99 72.39) (xy 154.94 72.39)
 		)
 		(stroke
@@
 			)
 			(justify right bottom)
+		)
+	)
+	(label "light"
+		(at 156.21 68.58 0)
+		(effects
+			(font
+				(size 1.27 1.27)
+			)
+			(justify left bottom)
 		)
 	)
@@
 	(symbol
 		(lib_id "power:+3.3V")
-		(at 191.77 64.77 90)
+		(at 173.99 64.77 90)
 		(unit 1)
 		(exclude_from_sim no)
@@
 		(dnp no)
 		(property "Reference" "#PWR03"
-			(at 195.58 64.77 0)
+			(at 177.8 64.77 0)
 			(effects
 				(font
@@
 		)
 		(property "Value" "+3.3V"
-			(at 187.96 64.7699 90)
+			(at 170.18 64.7699 90)
 			(effects
 				(font
@@
 		)
 		(property "Footprint" ""
-			(at 191.77 64.77 0)
+			(at 173.99 64.77 0)
 			(effects
 				(font
@@
 		)
 		(property "Datasheet" ""
-			(at 191.77 64.77 0)
+			(at 173.99 64.77 0)
 			(effects
 				(font
@@
 		)
 		(property "Description" "Power symbol creates a global label with name \"+3.3V\""
-			(at 191.77 64.77 0)
-			(effects
-				(font
+			(at 173.99 64.77 0)
+			(effects
+				(font
