File: PCB/sensor-board-solar/sensor-board-solar.kicad_pcb (KiCad board)
At the start: 2 copper layers, 23.6 x 23.5 mm, 7 parts, among them J1 Conn_01x02_Pin (Solar panel c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, U1 MAGNETIC POGO CONN., U2 MAGNETIC POGO CONN.

Commit message: Update PCB files (pressure + solar)#
Parts:
- added G***: LOGO, LOGO, B.Cu at (137.7, 97.2)
- moved R2 20.5 mm to (135.2, 97.7), turned to 180 degrees
- moved R3 18.7 mm to (140.2, 97.7), turned to 0 degrees
- moved R1 11.5 mm to (133.0, 89.7)
- moved H1 11.5 mm to (137.7, 103.8)
- moved U2 10.1 mm to (128.0, 93.1)
- moved U1 9.45 mm to (147.4, 93.1)
- moved J1 6.08 mm to (138.5, 90.3)
Connections:
- U1 pad 1: unconnected-(U1-Pad1) -> +3.3V
Routing:
- net +3.3V: track 7.84 -> 22.7 mm
- net GND: track 14.6 -> 0.00 mm
- net /ADC: track 10.2 -> 15.8 mm
- net Net-(J1-Pin_1): track 5.92 -> 9.14 mm
- added copper zone on B.Cu, net GND
- added copper zone on F.Cu, net GND
Other:
- board size 23.6 x 23.5 mm -> 30 x 28.1 mm
- board text added: "BOREALIS"
- board text added: "VOLTMETER"
- board text removed: "Borealis Voltmeter"

Commit message: made some changes
Parts:
- moved H1 0.06 mm to (137.7, 103.7)
Changed lines of the file:
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@@
 	(footprint "MountingHole:MountingHole_2.7mm_M2.5_Pad"
 		(layer "F.Cu")
-		(at 137.705 103.8)
+		(at 137.705 103.74)
 		(descr "Mounting Hole 2.7mm, M2.5, generated by kicad-footprint-generator mountinghole.py")
 		(tags "mountinghole M2.5")
@@
 		(polygon
 			(pts
-				(xy 112.92 72.32) (xy 157.99 71.41) (xy 157.41 112.45) (xy 119.05 109.39)
-			)
-		)
+				(xy 114.03 74.41) (xy 154.76 73.78) (xy 158.07 111.11) (xy 116.47 109.06)
+			)
+		)
