File: PCB/sensor-board-ozone/sensor-board-ozone.kicad_sch (KiCad schematic)
At the start: 6 parts, among them J2 Conn_01x04_Pin (MQ series sen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, J4 878-22-004-10-011101, J7 878-22-004-10-011101

Commit message: made some changes
Parts:
- removed J4, J7: 878-22-004-10-011101, BOREALIS:8782200410011101, symbol 878-22-004-10-011101:878-22-004-10-011101
- added U2, U3: MAGNETIC POGO CONN., batteryholder:MAGNETIC POGO CONN., symbol magnetic_pogo_conn.:MAGNETIC_POGO_CONN.
- J2: footprint (none) -> Connector_PinHeader_2.54mm:PinHeader_1x04_P2.54mm_Vertical
Connections:
- net +3.3V: now also U2.1, U3.2
- net +5V: now also U3.3
- net ADC: now also U2.2
- net GND: now also U3.1
- net ID: now also U3.4
- net SCL: now also U2.4
- net SDA: now also U2.3
- no-connect marks 2 -> 1
