File: PCB/sensor-board-ozone/sensor-board-ozone.kicad_pcb (KiCad board)
At the start: 2 copper layers, 30 x 28.2 mm, 8 parts, among them J2 Conn_01x04_Pin (MQ series sen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, U1 MAGNETIC POGO CONN., U2 MAGNETIC POGO CONN.

Commit message: Made some final checks and changes
Other:
- board text added: "GAS SENSOR"
- board text removed: "Gas Sensor"
Changed lines of the file:
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@@
 			(at 0 2.38 90)
 			(layer "B.SilkS")
+			(hide yes)
 			(effects
 				(font
@@
 		)
 	)
-	(gr_text "Gas Sensor"
+	(gr_text "GAS SENSOR"
 		(at 122.274998 59.979998 0)
 		(layer "B.SilkS" knockout)
