File: PCB/sensor-board-pressure/sensor-board-pressure.kicad_sch (KiCad schematic)
At the start: 9 parts, among them U1 MAGNETIC POGO CONN., U2 MAGNETIC POGO CONN.

Commit message: made some changes
Connections:
- net +3.3V: now also U1.1
- no-connect marks 2 -> 1
Other:
- moved on the sheet: U1, U2
