File: PCB/sensor-board-CO2-PA/sensor-board-CO2-PA.kicad_sch (KiCad schematic)
At the start: 8 parts, among them U1 SCD40-D-R2, U2 MAGNETIC POGO CONN., U3 MAGNETIC POGO CONN.

Commit message: made some changes
Parts:
- renumbered C5 to C1
Connections:
- net +3.3V: now also U2.1
- no-connect marks 15 -> 14
Other:
- moved on the sheet: U3

Commit message: Made some final checks and changes
Parts:
- added C2: 0.1uf, Capacitor_SMD:C_0805_2012Metric, symbol 2026-01-23_05-30-51:C0603C104K5RACTU
- C1: value 10microf -> 10uf
Connections:
- net +3.3V: now also C2.2
- net GND: now also C2.1
Changed lines of the file:
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@@
+	)
+	(junction
+		(at 90.17 48.26)
+		(diameter 0)
+		(color 0 0 0 0)
 	)
 	(junction
@@
 	(wire
 		(pts
-			(xy 90.17 55.88) (xy 90.17 39.37)
+			(xy 90.17 55.88) (xy 90.17 48.26)
 		)
 		(stroke
@@
 	(wire
 		(pts
+			(xy 114.3 48.26) (xy 123.19 48.26)
+		)
+		(stroke
+			(width 0)
+			(type default)
+		)
+	)
+	(wire
+		(pts
 			(xy 140.97 72.39) (xy 146.05 72.39)
 		)
@@
 	(wire
 		(pts
+			(xy 90.17 48.26) (xy 106.68 48.26)
+		)
+		(stroke
+			(width 0)
+			(type default)
+		)
+	)
+	(wire
+		(pts
 			(xy 48.26 55.88) (xy 62.23 55.88)
 		)
@@
 		(pts
 			(xy 62.23 49.53) (xy 62.23 55.88)
+		)
+		(stroke
+			(width 0)
+			(type default)
+		)
+	)
+	(wire
+		(pts
+			(xy 90.17 39.37) (xy 90.17 48.26)
 		)
 		(stroke
@@
 	)
 	(symbol
+		(lib_id "2026-01-23_05-30-51:C0603C104K5RACTU")
+		(at 114.3 48.26 180)
+		(unit 1)
+		(exclude_from_sim no)
+		(in_bom yes)
+		(on_board yes)
+		(dnp no)
+		(fields_autoplaced yes)
+		(property "Reference" "C2"
+			(at 110.49 41.91 0)
+			(effects
+				(font
+					(size 1.524 1.524)
+				)
+			)
+		)
+		(property "Value" "0.1uf"
+			(at 110.49 44.45 0)
+			(effects
+				(font
+					(size 1.524 1.524)
+				)
+			)
+		)
+		(property "Footprint" "Capacitor_SMD:C_0805_2012Metric"
+			(at 114.3 48.26 0)
+			(effects
+				(font
+					(size 1.27 1.27)
+					(italic yes)
+				)
+				(hide yes)
+			)
+		)
+		(property "Datasheet" "https://content.kemet.com/datasheets/KEM_C1002_X7R_SMD.pdf"
+			(at 114.3 48.26 0)
+			(effects
+				(font
+					(size 1.27 1.27)
+					(italic yes)
+				)
+				(hide yes)
+			)
+		)
+		(property "Description" ""
+			(at 114.3 48.26 0)
+			(effects
+				(font
+					(size 1.27 1.27)
+				)
+				(hide yes)
+			)
+		)
+		(pin "1"
+		)
+		(pin "2"
+		)
+		(instances
+			(project "sensor-board-CO2-PA"
+				(path "/4dc67bc0-6b27-441a-860a-e697f5d15d5c"
+					(reference "C2")
+					(unit 1)
+				)
+			)
+		)
+	)
+	(symbol
+		(lib_id "power:GND")
+		(at 123.19 48.26 90)
+		(unit 1)
+		(exclude_from_sim no)
+		(in_bom yes)
+		(on_board yes)
+		(dnp no)
+		(fields_autoplaced yes)
+		(property "Reference" "#PWR08"
+			(at 129.54 48.26 0)
+			(effects
+				(font
+					(size 1.27 1.27)
+				)
+				(hide yes)
+			)
+		)
+		(property "Value" "GND"
+			(at 127 48.2599 90)
+			(effects
+				(font
+					(size 1.27 1.27)
+				)
+				(justify right)
+			)
+		)
+		(property "Footprint" ""
+			(at 123.19 48.26 0)
+			(effects
+				(font
+					(size 1.27 1.27)
+				)
+				(hide yes)
+			)
+		)
+		(property "Datasheet" ""
+			(at 123.19 48.26 0)
+			(effects
+				(font
+					(size 1.27 1.27)
+				)
+				(hide yes)
+			)
+		)
+		(property "Description" "Power symbol creates a global label with name \"GND\" , ground"
+			(at 123.19 48.26 0)
+			(effects
+				(font
+					(size 1.27 1.27)
+				)
+				(hide yes)
+			)
+		)
+		(pin "1"
+		)
+		(instances
+			(project "sensor-board-CO2-PA"
+				(path "/4dc67bc0-6b27-441a-860a-e697f5d15d5c"
+					(reference "#PWR08")
+					(unit 1)
+				)
+			)
+		)
+	)
+	(symbol
 		(lib_id "power:+3.3V")
 		(at 139.7 92.71 0)
@@
 			)
 		)
-		(property "Value" "10microf"
+		(property "Value" "10uf"
 			(at 110.49 31.75 0)
 			(effects
