File: PCB/sensor-board-IMU/sensor-board-IMU.kicad_sch (KiCad schematic)
At the start: 5 parts, among them J4 878-22-004-10-011101, J7 878-22-004-10-011101

Commit message: Made some final checks and changes
Parts:
- removed J4, J7: 878-22-004-10-011101, BOREALIS:8782200410011101, symbol 878-22-004-10-011101:878-22-004-10-011101
- added C1: 0.1uF, Capacitor_SMD:C_0805_2012Metric, symbol 2026-01-23_05-30-51:C0603C104K5RACTU
- added C2: 10nF, Capacitor_SMD:C_0805_2012Metric, symbol 2026-01-23_05-30-51:C0603C104K5RACTU
- added H1: MountingHole, MountingHole:MountingHole_2.7mm_M2.5_Pad, symbol Mechanical:MountingHole
- added R2, R3: 4.7k, Resistor_SMD:R_0805_2012Metric, symbol Device:R
- added U2, U3: MAGNETIC POGO CONN., batteryholder:MAGNETIC POGO CONN., symbol magnetic_pogo_conn.:MAGNETIC_POGO_CONN.
- C5: value 100nF -> 0.1uf; footprint BOREALIS:CAPC17595_95N_KEM -> Capacitor_SMD:C_0805_2012Metric
- MPU6500: footprint (none) -> batteryholder:mpu6500
Connections:
- net +3.3V: now also C2.1, R2.1, R3.1, U2.1, U3.2
- net +5V: now also U3.3
- net ADC: now also U2.2
- net GND: now also MPU6500.11 (FSYNC), MPU6500.20 (RESV), C1.2, C2.2, U3.1
- net ID: now also U3.4
- net SCL: now also R2.2, U2.4
- net SDA: now also R3.2, U2.3
- net at MPU6500.10 (REGOUT): now also C1.1
- no-connect marks 1 -> 14
Other:
- moved on the sheet: C5
