File: PCB/sensor-board-light/sensor-board-light.kicad_pcb (KiCad board)
At the start: 2 copper layers, 30.9 x 38 mm, 13 parts, among them J1 Conn_01x04_Pin, J3 Conn_01x04_Pin, U1 MAGNETIC POGO CONN., U2 MAGNETIC POGO CONN.

Commit message: made some changes
Parts:
- added G***: LOGO, LOGO, B.Cu at (164.8, 82.6)
- J3: footprint Connector_PinHeader_2.54mm:PinHeader_1x04_P2.54mm_Vertical -> Connector_JST:JST_PH_B4B-PH-K_1x04_P2.00mm_Vertical
- moved H3 45.2 mm to (167.5, 112.3)
- moved H2 44.8 mm to (167.5, 105.3)
- moved LTR-390UV-01 34.4 mm to (162.5, 109.5), turned to 0 degrees
- moved C1 32.3 mm to (156.2, 117.1), turned to 0 degrees
- moved R6 30.0 mm to (168.9, 81.0), turned to 90 degrees
- moved J3 29.3 mm to (155.6, 112.8), turned to 90 degrees
- moved U1 25.0 mm to (174.6, 78.5)
- moved H1 24.7 mm to (164.9, 89.2)
- moved J1 23.6 mm to (168.0, 75.7)
- moved R3 23.4 mm to (155.8, 102.0), turned to 0 degrees
- moved U2 22.8 mm to (155.3, 78.5)
- moved R1 22.5 mm to (161.0, 70.7)
- moved R5 17.4 mm to (160.9, 81.1), turned to 90 degrees
Connections:
- U1 pad 1: unconnected-(U1-Pad1) -> +3.3V
Routing:
- net +3.3V: track 23.8 -> 54.6 mm, vias 0 -> 1
- net /SDA: track 14.7 -> 29.7 mm, vias 1 -> 0
- net GND: track 23.9 -> 13.3 mm
- net Net-(LTR-390UV-01-INT): track 7.63 -> 11.8 mm
- net /3.3v: track 22.7 -> 26.8 mm
- net /SCL1: track 12.3 -> 8.46 mm
- net /SDA1: track 9.02 -> 6.35 mm
- net /ID: track 4.54 -> 6.79 mm
- net /SCL: track 17.8 -> 17.5 mm, vias 1 -> 0
- added copper zone on B.Cu, net GND
- added copper zone on F.Cu, net GND
Other:
- board size 30.9 x 38 mm -> 30 x 55.1 mm
- board text added: "BOREALIS"
- board text added: "Light Sensor"
- board text removed: "Borealis Light Sensor"
- board text removed: "External light sensor module"

Commit message: Made some final checks and changes
Parts:
- added C2: 4.7uF, Capacitor_SMD:C_0805_2012Metric, F.Cu at (154.0, 120.0)
- C1: value 100nF -> 0.1uF
- moved H3 5.85 mm to (165.9, 117.9)
- moved C1 4.09 mm to (159.1, 120.0)
- moved J3 3.47 mm to (153.8, 115.8)
- moved R3 3.47 mm to (154.1, 105.0)
- moved U1 3.47 mm to (172.8, 81.5)
- moved G*** 3.47 mm to (163.1, 85.6)
- moved H1 3.47 mm to (163.2, 92.2)
- moved R1 3.47 mm to (159.3, 73.7)
- moved R6 3.47 mm to (167.1, 84.0)
- moved U2 3.47 mm to (153.5, 81.5)
- moved J1 3.47 mm to (166.3, 78.7)
- moved LTR-390UV-01 3.47 mm to (160.7, 112.4)
- moved R5 3.47 mm to (159.1, 84.1)
- moved H2 2.36 mm to (165.8, 107.0)
Routing:
- net /3.3v: track 26.8 -> 37.1 mm
- net GND: track 13.3 -> 21.3 mm
Other:
- outline, holes or cut-outs redrawn
- board text added: "LIGHT SENSOR"
- board text removed: "Light Sensor"
