File: PCB/sensor-board-light/sensor-board-light.kicad_sch (KiCad schematic)
At the start: 13 parts, among them J1 Conn_01x04_Pin, J3 Conn_01x04_Pin, U2 MAGNETIC POGO CONN., U3 MAGNETIC POGO CONN.

Commit message: made some changes
Parts:
- J3: footprint Connector_PinHeader_2.54mm:PinHeader_1x04_P2.54mm_Vertical -> Connector_JST:JST_PH_B4B-PH-K_1x04_P2.00mm_Vertical
Connections:
- net +3.3V: now also U2.1
- no-connect marks 2 -> 1
Other:
- moved on the sheet: U3

Commit message: Made some final checks and changes
Parts:
- added C2: 4.7uF, Capacitor_SMD:C_0805_2012Metric, symbol 2026-01-23_05-30-51:C0603C104K5RACTU
- C1: value 100nF -> 0.1uF
Connections:
- net 3.3v: now also C2.2
- net GND: now also C2.1
Other:
- moved on the sheet: C1
Changed lines of the file:
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@@
 	(paper "A4")
 	(rectangle
-		(start 22.86 27.94)
+		(start 15.24 27.94)
 		(end 92.71 77.47)
 		(stroke
@@
 	)
 	(junction
-		(at 30.48 66.04)
+		(at 27.94 66.04)
+		(diameter 0)
+		(color 0 0 0 0)
+	)
+	(junction
+		(at 27.94 73.66)
 		(diameter 0)
 		(color 0 0 0 0)
@@
 	)
 	(junction
+		(at 21.59 73.66)
+		(diameter 0)
+		(color 0 0 0 0)
+	)
+	(junction
 		(at 163.83 55.88)
 		(diameter 0)
@@
 	)
 	(junction
-		(at 30.48 73.66)
+		(at 21.59 66.04)
 		(diameter 0)
 		(color 0 0 0 0)
@@
 	(wire
 		(pts
+			(xy 27.94 66.04) (xy 33.02 66.04)
+		)
+		(stroke
+			(width 0)
+			(type default)
+		)
+	)
+	(wire
+		(pts
 			(xy 138.43 104.14) (xy 125.73 104.14)
 		)
@@
 	(wire
 		(pts
+			(xy 21.59 73.66) (xy 27.94 73.66)
+		)
+		(stroke
+			(width 0)
+			(type default)
+		)
+	)
+	(wire
+		(pts
 			(xy 144.78 59.69) (xy 146.05 59.69)
 		)
@@
 	(wire
 		(pts
+			(xy 21.59 66.04) (xy 27.94 66.04)
+		)
+		(stroke
+			(width 0)
+			(type default)
+		)
+	)
+	(wire
+		(pts
 			(xy 128.27 107.95) (xy 128.27 110.49)
 		)
@@
 	(wire
 		(pts
-			(xy 30.48 73.66) (xy 39.37 73.66)
-		)
-		(stroke
-			(width 0)
-			(type default)
-		)
-	)
-	(wire
-		(pts
 			(xy 57.15 68.58) (xy 82.55 68.58)
 		)
@@
 	(wire
 		(pts
-			(xy 25.4 73.66) (xy 30.48 73.66)
+			(xy 16.51 73.66) (xy 21.59 73.66)
 		)
 		(stroke
@@
 	(wire
 		(pts
+			(xy 27.94 73.66) (xy 39.37 73.66)
+		)
+		(stroke
+			(width 0)
+			(type default)
+		)
+	)
+	(wire
+		(pts
 			(xy 163.83 55.88) (xy 163.83 63.5)
 		)
@@
 	(wire
 		(pts
-			(xy 25.4 66.04) (xy 30.48 66.04)
+			(xy 16.51 66.04) (xy 21.59 66.04)
 		)
 		(stroke
@@
 		(pts
 			(xy 149.86 106.68) (xy 149.86 109.22)
-		)
-		(stroke
-			(width 0)
-			(type default)
-		)
-	)
-	(wire
-		(pts
-			(xy 30.48 66.04) (xy 33.02 66.04)
 		)
 		(stroke
@@
 	)
 	(label "3.3v"
-		(at 25.4 66.04 0)
+		(at 16.51 66.04 0)
 		(effects
 			(font
@@
 	)
 	(label "GND"
-		(at 25.4 73.66 0)
+		(at 16.51 73.66 0)
 		(effects
 			(font
@@
 			)
 			(justify left bottom)
+		)
+	)
+	(symbol
+		(lib_id "2026-01-23_05-30-51:C0603C104K5RACTU")
+		(at 27.94 73.66 90)
+		(unit 1)
+		(exclude_from_sim no)
+		(in_bom yes)
+		(on_board yes)
+		(dnp no)
+		(property "Reference" "C2"
+			(at 31.75 68.5799 90)
+			(effects
+				(font
+					(size 1.524 1.524)
+				)
+				(justify right)
+			)
+		)
+		(property "Value" "4.7uF"
+			(at 29.21 75.184 90)
+			(effects
+				(font
+					(size 1.524 1.524)
+				)
+				(justify right)
+			)
+		)
+		(property "Footprint" "Capacitor_SMD:C_0805_2012Metric"
+			(at 27.94 73.66 0)
+			(effects
+				(font
+					(size 1.27 1.27)
+					(italic yes)
+				)
+				(hide yes)
+			)
+		)
+		(property "Datasheet" "https://content.kemet.com/datasheets/KEM_C1002_X7R_SMD.pdf"
+			(at 27.94 73.66 0)
+			(effects
+				(font
+					(size 1.27 1.27)
+					(italic yes)
+				)
+				(hide yes)
+			)
+		)
+		(property "Description" ""
+			(at 27.94 73.66 0)
+			(effects
+				(font
+					(size 1.27 1.27)
+				)
+				(hide yes)
+			)
+		)
+		(pin "1"
+		)
+		(pin "2"
+		)
+		(instances
+			(project "sensor-board-light"
+				(path "/726314c5-8b2a-4d92-8d4d-3d9717bee1d8"
+					(reference "C2")
+					(unit 1)
+				)
+			)
 		)
 	)
@@
 	(symbol
 		(lib_id "2026-01-23_05-30-51:C0603C104K5RACTU")
-		(at 30.48 73.66 90)
+		(at 21.59 73.66 90)
 		(unit 1)
 		(exclude_from_sim no)
@@
 		(on_board yes)
 		(dnp no)
-		(fields_autoplaced yes)
 		(property "Reference" "C1"
-			(at 34.29 68.5799 90)
+			(at 21.336 62.992 90)
 			(effects
 				(font
@@
 			)
 		)
-		(property "Value" "100nF"
-			(at 34.29 71.1199 90)
+		(property "Value" "0.1uF"
+			(at 19.05 75.946 90)
 			(effects
 				(font
@@
 		)
 		(property "Footprint" "Capacitor_SMD:C_0805_2012Metric"
-			(at 30.48 73.66 0)
+			(at 21.59 73.66 0)
 			(effects
 				(font
@@
 		)
 		(property "Datasheet" "https://content.kemet.com/datasheets/KEM_C1002_X7R_SMD.pdf"
-			(at 30.48 73.66 0)
+			(at 21.59 73.66 0)
 			(effects
 				(font
@@
 		)
 		(property "Description" ""
-			(at 30.48 73.66 0)
-			(effects
-				(font
+			(at 21.59 73.66 0)
+			(effects
+				(font
