File: PCB/sensor-board-magnetic-field/sensor-board-magnetic-field.kicad_pcb (KiCad board)
At the start: 2 copper layers, 23.6 x 23.5 mm, 8 parts, among them U1 MAGNETIC POGO CONN., U2 MAGNETIC POGO CONN.

Commit message: made some changes
Parts:
- added G***: LOGO, LOGO, B.Cu at (141.7, 108.2)
- moved R2 26.0 mm to (146.2, 103.0), turned to 180 degrees
- moved U1 24.0 mm to (151.3, 104.7)
- moved H1 23.2 mm to (141.7, 115.4)
- moved TLV493D1 22.7 mm to (141.5, 101.8)
- moved U2 21.7 mm to (132.0, 104.7)
- moved R1 21.2 mm to (137.2, 100.0)
- moved R3 20.7 mm to (137.4, 103.5), turned to 0 degrees
- moved C5 19.5 mm to (136.8, 108.0), turned to 90 degrees
Connections:
- U1 pad 1: unconnected-(U1-Pad1) -> +3.3V
Routing:
- net GND: track 24.5 -> 3.34 mm, vias 1 -> 0
- net +3.3V: track 24.9 -> 34.2 mm, vias 4 -> 1
- net /SCL: track 15.2 -> 18.1 mm
- net /SDA: track 9.83 -> 10.7 mm
- net /ID: track 4.86 -> 5.37 mm
- added copper zone on B.Cu, net GND
- added copper zone on F.Cu, net GND
Other:
- board size 23.6 x 23.5 mm -> 30 x 28.1 mm
- board text added: "BOREALIS"
- board text added: "Magnetometer"
- board text removed: "Borealis Magnetometer"

Commit message: Made some final checks and changes
Parts:
- removed TLV493D1: ~, batteryholder:TLV493D
- added MMC5603NJ1: ~, batteryholder:XDCR_MMC5603NJ, B.Cu at (138.0, 72.9)
- C5: value 100nF -> 2.2uf
- R2, R3: value 10K -> 2.7k
- moved C5 33.0 mm to (134.6, 75.1)
- moved R2 32.1 mm to (142.2, 71.2), turned to 0 degrees
- moved R1 29.3 mm to (134.7, 70.8)
- moved U1 29.1 mm to (147.7, 75.8)
- moved U2 29.1 mm to (128.4, 75.8)
- moved H1 29.1 mm to (138.1, 86.5)
- moved G*** 29.1 mm to (138.0, 79.3)
- moved R3 29.1 mm to (142.1, 74.9)
Connections:
- R2 pad 1: +3.3V -> /SDA
- R2 pad 2: /SDA -> +3.3V
- R3 pad 1: +3.3V -> /SCL
- R3 pad 2: /SCL -> +3.3V
Routing:
- net GND: track 3.34 -> 22.0 mm
- net /SCL: track 18.1 -> 13.0 mm
- net /SDA: track 10.7 -> 15.1 mm
- net +3.3V: track 34.2 -> 32.3 mm
- net /ID: track 5.37 -> 7.12 mm
Other:
- board text added: "MAGNETOMETER"
- board text removed: "Magnetometer"
