File: PCB/sensor-board-magnetic-field/sensor-board-magnetic-field.kicad_sch (KiCad schematic)
At the start: 8 parts, among them U2 MAGNETIC POGO CONN., U3 MAGNETIC POGO CONN.

Commit message: made some changes
Connections:
- net +3.3V: now also U2.1
- no-connect marks 1 -> 0
Other:
- moved on the sheet: U3

Commit message: Made some final checks and changes
Parts:
- removed TLV493D1: ~, batteryholder:TLV493D, symbol TLV493DA1B6HTSA2_2025-12-27-altium-import:root_0_TLV493DA1B6HTSA2_
- added MMC5603NJ1: ~, batteryholder:XDCR_MMC5603NJ, symbol MMC5603NJ_2026-02-16-altium-import:root_0_MMC5603NJ_
- C5: value 100nF -> 2.2uf
- R2, R3: value 10K -> 2.7k
Connections:
- net +3.3V: now also R2.2, R3.2, MMC5603NJ1.B1 (VDD); no longer R2.1, R3.1
- net GND: now also MMC5603NJ1.A1 (VSA)
- net SCL: now also R3.1, MMC5603NJ1.A2 (SCL); no longer R3.2
- net SDA: now also R2.1, MMC5603NJ1.B2 (SDA); no longer R2.2
Other:
- moved on the sheet: C5
